File: starter-ortho.kicad_pcb (KiCad board)
At the start: 2 copper layers, 272.3 x 82.6 mm, 98 parts, among them SW1 SW_Push, U1 ProMicro

Commit message: Added silkscreen text for promicro (and other updates)
Routing:
- net COL0: track 177.8 -> 192.9 mm
- net COL1: track 160.5 -> 174.1 mm
- net COL4: track 110.7 -> 113.0 mm
- net COL5: track 92.3 -> 94.4 mm
- net COL3: track 129.5 -> 131.6 mm
- net COL2: track 149.6 -> 151.5 mm
Other:
- board text added: "Electronics face down!"
- board text removed: "Split-ish Ortho"
